Commit message: Minor fixes

File: src/ur_onrobot/ur_onrobot_moveit_config/srdf/ur_onrobot_macro.srdf.xacro (robot description, xacro)
@@ -69,10 +69,10 @@
     </group_state>
     <group_state name="${prefix}ready_pose2" group="${prefix}${name}_manipulator">
-      <joint name="${prefix}elbow_joint" value="-0.27" />
-      <joint name="${prefix}shoulder_lift_joint" value="-2.14" />
-      <joint name="${prefix}shoulder_pan_joint" value="-1.23" />
-      <joint name="${prefix}wrist_1_joint" value="-2.27" />
-      <joint name="${prefix}wrist_2_joint" value="1.54" />
-      <joint name="${prefix}wrist_3_joint" value="-0.11" />
+      <joint name="${prefix}shoulder_pan_joint" value="-0.82" />
+      <joint name="${prefix}wrist_3_joint" value="0.74" />
+      <joint name="${prefix}wrist_2_joint" value="1.57" />
+      <joint name="${prefix}wrist_1_joint" value="-2.24" />
+      <joint name="${prefix}elbow_joint" value="-0.66" />
+      <joint name="${prefix}shoulder_lift_joint" value="-1.8" />
     </group_state>
     <!--END EFFECTOR - Purpose - Represent information about an end effector.-->

Commit message: Fixes

File: src/ur_onrobot/ur_onrobot_moveit_config/srdf/ur_onrobot_macro.srdf.xacro (robot description, xacro)
@@ -75,4 +75,12 @@
       <joint name="${prefix}elbow_joint" value="-0.66" />
       <joint name="${prefix}shoulder_lift_joint" value="-1.8" />
+    </group_state>
+    <group_state name="${prefix}search" group="${prefix}${name}_manipulator">
+      <joint name="${prefix}shoulder_pan_joint" value="-1.24" />
+      <joint name="${prefix}wrist_3_joint" value="0.32" />
+      <joint name="${prefix}wrist_2_joint" value="1.57" />
+      <joint name="${prefix}wrist_1_joint" value="-2.53" />
+      <joint name="${prefix}elbow_joint" value="-0.66" />
+      <joint name="${prefix}shoulder_lift_joint" value="-1.51" />
     </group_state>
     <!--END EFFECTOR - Purpose - Represent information about an end effector.-->

Commit message: Final

File: src/ur_onrobot/ur_onrobot_moveit_config/srdf/ur_onrobot_macro.srdf.xacro (robot description, xacro)
@@ -77,10 +77,10 @@
     </group_state>
     <group_state name="${prefix}search" group="${prefix}${name}_manipulator">
-      <joint name="${prefix}shoulder_pan_joint" value="-1.24" />
+      <joint name="${prefix}shoulder_pan_joint" value="-1.23" />
       <joint name="${prefix}wrist_3_joint" value="0.32" />
       <joint name="${prefix}wrist_2_joint" value="1.57" />
-      <joint name="${prefix}wrist_1_joint" value="-2.53" />
-      <joint name="${prefix}elbow_joint" value="-0.66" />
-      <joint name="${prefix}shoulder_lift_joint" value="-1.51" />
+      <joint name="${prefix}wrist_1_joint" value="-2.78" />
+      <joint name="${prefix}elbow_joint" value="-0.21" />
+      <joint name="${prefix}shoulder_lift_joint" value="-1.70" />
     </group_state>
     <!--END EFFECTOR - Purpose - Represent information about an end effector.-->
